Commit message: Updated MoveIt configuration for HC20DTP robot

File: hc20_moveit_config/config/motoman_hc20.urdf.xacro (robot description, xacro)
@@ -1,4 +1,4 @@
 <?xml version="1.0"?>
-<robot xmlns:xacro="http://www.ros.org/wiki/xacro" name="motoman_hc10dt">
+<robot xmlns:xacro="http://www.ros.org/wiki/xacro" name="motoman_hc20">
     <xacro:arg name="initial_positions_file" default="initial_positions.yaml" />
     <!-- Import motoman_hc20 urdf file -->

File: hc20_moveit_config/urdf/hc20.urdf (robot description, URDF)
Before this commit: robot motoman_hc20, 10 links, 9 joints
Links:
- link base_link: geometry collision mesh filename=package://hc20_moveit_config/meshes/collision/base_link.stl; visual mesh filename=package://hc20_moveit_config/meshes/visual/base_link.stl
- link link_5: geometry collision mesh filename=package://hc20_moveit_config/meshes/collision/link_5_b.stl; visual mesh filename=package://hc20_moveit_config/meshes/visual/link_5_b.dae
- link link_6: geometry collision mesh filename=package://hc20_moveit_config/meshes/collision/link_6_t.stl; visual mesh filename=package://hc20_moveit_config/meshes/visual/link_6_t.dae
Joints:
- joint joint_1: limit lower=-3.141592653589793 upper=3.141592653589793 effort=368.48 velocity=2.2689280275926285 -> lower=${radians(-210)} upper=${radians(210)} effort=917.28 velocity=${radians(80)}
- joint joint_2: limit lower=-3.141592653589793 upper=3.141592653589793 effort=368.48 velocity=2.2689280275926285 -> lower=${radians(-180)} upper=${radians(180)} effort=1223.04 velocity=${radians(80)}
- joint joint_3: limit lower=-0.08726646259971647 upper=6.19591884457987 effort=141.12 velocity=3.141592653589793 -> lower=${radians(-67)} upper=${radians(247)} effort=642.88 velocity=${radians(120)}
- joint joint_4: limit lower=-3.141592653589793 upper=3.141592653589793 effort=39.20 velocity=3.141592653589793 -> lower=${radians(-210)} upper=${radians(210)} effort=368.48 velocity=${radians(130)}
- joint joint_5: limit lower=-3.141592653589793 upper=3.141592653589793 effort=31.36 velocity=4.363323129985824 -> lower=${radians(-180)} upper=${radians(180)} effort=141.12 velocity=${radians(180)}
- joint joint_6: limit lower=-3.141592653589793 upper=3.141592653589793 effort=31.36 velocity=4.363323129985824 -> lower=${radians(-210)} upper=${radians(210)} effort=141.12 velocity=${radians(180)}

File: hc20_moveit_config/urdf/hc20_macro.xacro (robot description, xacro)
@@ -7,5 +7,5 @@
       <visual>
         <geometry>
-          <mesh filename="package://hc20_moveit_config/meshesvisual/base_link.stl"/>
+          <mesh filename="package://hc20_moveit_config/meshes/visual/base_link.stl"/>
         </geometry>
         <xacro:material_yaskawa_blue/>
@@ -72,5 +72,5 @@
       <visual>
         <geometry>
-          <mesh filename="package://hc20_moveit_config/meshes/visual/link_5_b.stl"/>
+          <mesh filename="package://hc20_moveit_config/meshes/visual/link_5_b.dae"/>
         </geometry>
         <xacro:material_yaskawa_blue/>
@@ -85,5 +85,5 @@
       <visual>
         <geometry>
-          <mesh filename="package://hc20_moveit_config/meshes/visual/link_6_t.stl"/>
+          <mesh filename="package://hc20_moveit_config/meshes/visual/link_6_t.dae"/>
         </geometry>
         <xacro:material_yaskawa_blue/>
@@ -103,5 +103,5 @@
       <origin xyz="0 0 0.380" rpy="0 0 0" />
       <axis xyz="0 0 1" />
-      <limit lower="${radians(-180)}" upper="${radians(180)}" effort="917.28" velocity="${radians(80)}"/>
+      <limit lower="${radians(-210)}" upper="${radians(210)}" effort="917.28" velocity="${radians(80)}"/>
     </joint>
     <joint name="${prefix}joint_2" type="revolute">
