Commit message: Liner move works on the robot.

File: hc10_movit2v3/config/motoman_hc10dt.urdf.xacro (robot description, xacro)
@@ -5,5 +5,5 @@
     <xacro:include filename="$(find hc10dt_moveit_config)/urdf/hc10dt.urdf" />
     <!-- Import control_xacro -->
-    <xacro:include filename="motoman_hc10dt.ros2_control.xacro" />
-    <xacro:motoman_hc10dt_ros2_control name="FakeSystem" initial_positions_file="$(arg initial_positions_file)"/>
+    <!-- <xacro:include filename="motoman_hc10dt.ros2_control.xacro" />
+    <xacro:motoman_hc10dt_ros2_control name="FakeSystem" initial_positions_file="$(arg initial_positions_file)"/> -->
 </robot>

File: hc10dt_moveit_config/config/motoman_hc10dt.urdf.xacro (robot description, xacro)
@@ -4,6 +4,7 @@
     <!-- Import motoman_hc10dt urdf file -->
     <xacro:include filename="$(find hc10dt_moveit_config)/urdf/hc10dt.urdf" />
+    <!-- <xacro:include filename="$(find hc10dt_moveit_config)/config/motoman_hc10dt.ros2_control.xacro" /> -->
     <!-- Import control_xacro -->
-    <xacro:include filename="motoman_hc10dt.ros2_control.xacro" />
+    <!-- <xacro:include filename="motoman_hc10dt.ros2_control.xacro" /> -->
     <!-- <xacro:motoman_hc10dt_ros2_control name="FakeSystem" initial_positions_file="$(arg initial_positions_file)"/> -->
 </robot>

File: hc10dt_moveit_config/urdf/hc10dt.urdf (robot description, URDF)
Before this commit: robot motoman_hc10dt, 9 links, 8 joints
Links:
- added link world
Joints:
- added joint world_to_base_link: type fixed, parent world, child base_link, origin xyz=0 0 0.275 rpy=0 0 0

Commit message: Simulation for HC20DTP

File: hc10_movit2v3/config/motoman_hc10dt.urdf.xacro (robot description, xacro)
@@ -5,5 +5,5 @@
     <xacro:include filename="$(find hc10dt_moveit_config)/urdf/hc10dt.urdf" />
     <!-- Import control_xacro -->
-    <!-- <xacro:include filename="motoman_hc10dt.ros2_control.xacro" />
-    <xacro:motoman_hc10dt_ros2_control name="FakeSystem" initial_positions_file="$(arg initial_positions_file)"/> -->
+    <xacro:include filename="motoman_hc10dt.ros2_control.xacro" />
+    <xacro:motoman_hc10dt_ros2_control name="FakeSystem" initial_positions_file="$(arg initial_positions_file)"/>
 </robot>

File: hc20_sim_moveit_config/config/motoman_hc20_sim.ros2_control.xacro (robot description, xacro)
@@ -1,5 +1,5 @@
 <?xml version="1.0"?>
 <robot xmlns:xacro="http://www.ros.org/wiki/xacro">
-    <xacro:macro name="motoman_hc10dt_ros2_control" params="name initial_positions_file">
+    <xacro:macro name="motoman_hc20_sim_ros2_control" params="name initial_positions_file">
         <xacro:property name="initial_positions" value="${load_yaml(initial_positions_file)['initial_positions']}"/>
         <ros2_control name="${name}" type="system">
