Commit message: Final tunning

File: hc20_moveit_config/urdf/hc20.urdf (robot description, URDF)
Before this commit: robot motoman_hc20, 10 links, 9 joints
Joints:
- joint joint_1: limit lower=${radians(-210)} upper=${radians(210)} effort=917.28 velocity=${radians(80)} -> lower=-3.665191 upper=3.665191 effort=917.28 velocity=1.396263
- joint joint_2: limit lower=${radians(-180)} upper=${radians(180)} effort=1223.04 velocity=${radians(80)} -> lower=-3.141593 upper=3.141593 effort=1223.04 velocity=1.396263
- joint joint_3: limit lower=${radians(-67)} upper=${radians(247)} effort=642.88 velocity=${radians(120)} -> lower=-1.169371 upper=4.312240 effort=642.88 velocity=2.094395
- joint joint_4: limit lower=${radians(-210)} upper=${radians(210)} effort=368.48 velocity=${radians(130)} -> lower=-3.665191 upper=3.665191 effort=368.48 velocity=2.268928
- joint joint_5: limit lower=${radians(-180)} upper=${radians(180)} effort=141.12 velocity=${radians(180)} -> lower=-3.141593 upper=3.141593 effort=141.12 velocity=3.141593
- joint joint_6: limit lower=${radians(-210)} upper=${radians(210)} effort=141.12 velocity=${radians(180)} -> lower=-3.665191 upper=3.665191 effort=141.12 velocity=3.141593
- joint joint_6-tool0: origin xyz=0 0 -0.170 rpy=3.141592653589793 0 0 -> xyz=0.200 0 0 rpy=0 0 0
- joint world_to_base_link: origin xyz=0 0 0.380 rpy=0 0 0 -> xyz=0 0 -0.380 rpy=0 0 0
